File: PCB-Design/LED Control.kicad_pcb (KiCad board)
At the start: 2 copper layers, 60 x 80 mm, 28 parts, among them J1 5V 5A Power, J2 TO WS2812B LED STRIP, J3 Sound Sensor, SW1 SW_Push_Dual

Commit message: gerbers generated
Parts:
- J2, J3: footprint TerminalBlock_Phoenix:TerminalBlock_Phoenix_MPT-0,5-3-2.54_1x03_P2.54mm_Horizontal -> TerminalBlock_TE-Connectivity:TerminalBlock_TE_282834-3_1x03_P2.54mm_Horizontal
- moved R6 6.36 mm to (120.6, 125.4), turned to 90 degrees
- moved D4 3.35 mm to (115.8, 125.3), turned to 90 degrees
- moved C1 1.66 mm to (120.2, 118.0)
- moved C2 1.66 mm to (116.9, 118.0)
- moved C3 1.66 mm to (113.3, 118.0)
Routing:
- net VCC: track 0.00 -> 14.0 mm
- net GND: track 27.1 -> 36.9 mm
