File: PCB-Design/LED Control.sch (KiCad schematic (older format))
At the start: 24 parts, among them J1 5V 5A Power, J2 TO WS2812B LED STRIP, J3 Sound Sensor, SW1 SW_Push_Dual

Commit message: gerbers generated
Parts:
- J2, J3: footprint TerminalBlock_Phoenix:TerminalBlock_Phoenix_MPT-0,5-3-2.54_1x03_P2.54mm_Horizontal -> TerminalBlock_TE-Connectivity:TerminalBlock_TE_282834-3_1x03_P2.54mm_Horizontal
Changed lines of the file:
@@
 F 0 "J2" H 5218 2575 50  0000 C CNN
 F 1 "TO WS2812B LED STRIP" H 5218 2666 50  0000 C CNN
-F 2 "TerminalBlock_Phoenix:TerminalBlock_Phoenix_MPT-0,5-3-2.54_1x03_P2.54mm_Horizontal" H 5300 2900 50  0001 C CNN
+F 2 "TerminalBlock_TE-Connectivity:TerminalBlock_TE_282834-3_1x03_P2.54mm_Horizontal" H 5300 2900 50  0001 C CNN
 F 3 "~" H 5300 2900 50  0001 C CNN
 	1    5300 2900
@@
 F 0 "J3" H 1718 5175 50  0000 C CNN
 F 1 "Sound Sensor" H 1718 5266 50  0000 C CNN
-F 2 "TerminalBlock_Phoenix:TerminalBlock_Phoenix_MPT-0,5-3-2.54_1x03_P2.54mm_Horizontal" H 1800 5500 50  0001 C CNN
+F 2 "TerminalBlock_TE-Connectivity:TerminalBlock_TE_282834-3_1x03_P2.54mm_Horizontal" H 1800 5500 50  0001 C CNN
 F 3 "~" H 1800 5500 50  0001 C CNN
 	1    1800 5500
@@
 $EndComp
 Wire Wire Line
-	9350 2700 9800 2700
-Wire Wire Line
 	9500 3550 9800 3550
 Wire Wire Line
@@
 	9950 2200 10450 2200
 $Comp
-L power:GND #PWR?
+L power:GND #PWR0101
 U 1 1 5E621F08
 P 6100 2500
-F 0 "#PWR?" H 6100 2250 50  0001 C CNN
+F 0 "#PWR0101" H 6100 2250 50  0001 C CNN
 F 1 "GND" H 6105 2327 50  0000 C CNN
 F 2 "" H 6100 2500 50  0001 C CNN
@@
 Wire Wire Line
 	6100 2800 6100 2500
+Wire Wire Line
+	9800 2700 9350 2700
 $EndSCHEMATC
